Commit message: add joint controller plugins to gazebo

File: src/deman_simulation/description/gazebo.xacro (robot description, xacro)
@@ -13,3 +13,23 @@
         <material>Gazebo/Blue</material>
     </gazebo>
+    <gazebo reference="c_link">
+        <material>Gazebo/Yellow</material>
+    </gazebo>
+    <gazebo>
+        <plugin name="gazebo_ros_joint_state_publisher"
+            filename="libgazebo_ros_joint_state_publisher.so">
+            <update_rate>20</update_rate>
+            <joint_name>x_joint</joint_name>
+            <joint_name>y_joint</joint_name>
+            <joint_name>z_joint</joint_name>
+            <joint_name>c_joint</joint_name>
+        </plugin>
+    </gazebo>
+    <gazebo>
+        <plugin name="gazebo_ros_joint_pose_trajectory"
+            filename="libgazebo_ros_joint_pose_trajectory.so">
+            <update_rate>2</update_rate>
+        </plugin>
+    </gazebo>
+    <!-- rostopic pub -1 /set_joint_trajectory trajectory_msgs/msg/JointTrajectory  '{header: {frame_id: world}, joint_names: [x_joint, y_joint], points: [  {positions: {0.2,0.2}} ]}' -->
 </robot>

File: src/deman_simulation/description/include.xacro (robot description, xacro)
@@ -13,4 +13,7 @@
         <color rgba="0 1 0 1"/>
     </material>
+    <material name="yellow">
+        <color rgba="0.5 0.5 0 1"/>
+    </material>
     <xacro:macro name="inertial_box" params="mass x y z *origin">
         <inertial>
